File: hardware/BalloonPCB/BalloonPCB.kicad_pcb (KiCad board)
At the start: 2 copper layers, 76.2 x 76.2 mm, 15 parts, among them P1 BMP180_HEADER, P2 GPS_HEADER, P3 ACCEL_HEADER, P4 CONN_01X24, P5 CONN_01X24, P6 5VDC_HEADER, P7 SMA, P8 THERMO_HEADER, U1 Teensy3.5, U2 HX1

Commit message: Add prototyping section
Parts:
- added P10: CONN_01X04, Pin_Headers:Pin_Header_Straight_1x04_Pitch2.00mm, F.Cu at (121.9, 58.4)
- added P11: CONN_01X04, Pin_Headers:Pin_Header_Straight_1x04_Pitch2.00mm, F.Cu at (121.9, 55.9)
- added P9: CONN_01X04, Pin_Headers:Pin_Header_Straight_1x04_Pitch2.00mm, F.Cu at (121.9, 61.0)
Routing:
- net Net-(P10-Pad4): track 0.00 -> 5.08 mm
- net Net-(P10-Pad3): track 0.00 -> 5.08 mm
- net Net-(P10-Pad2): track 0.00 -> 5.08 mm
- net Net-(P10-Pad1): track 0.00 -> 5.08 mm
Changed lines of the file:
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@@
 (kicad_pcb (version 4) (host pcbnew 4.0.5)
   (general
-    (links 89)
-    (no_connects 1)
+    (links 97)
+    (no_connects 5)
     (area 50.672999 50.672999 127.127001 127.127001)
     (thickness 1.6)
     (drawings 11)
-    (tracks 145)
+    (tracks 153)
     (zones 0)
-    (modules 15)
-    (nets 62)
+    (modules 18)
+    (nets 66)
   )
   (page USLetter)
@@
     (mod_text_size 1 1)
     (mod_text_width 0.15)
-    (pad_size 1.7272 2.6)
-    (pad_drill 1.2)
+    (pad_size 1.35 1.016)
+    (pad_drill 0.8)
     (pad_to_mask_clearance 0.2)
     (aux_axis_origin 0 0)
@@
   (net 60 TXD)
   (net 61 RF+)
+  (net 62 "Net-(P10-Pad1)")
+  (net 63 "Net-(P10-Pad2)")
+  (net 64 "Net-(P10-Pad3)")
+  (net 65 "Net-(P10-Pad4)")
   (net_class Default "This is the default net class."
     (clearance 0.79375)
@@
     (add_net GPS_SDA)
     (add_net GPS_TXD)
+    (add_net "Net-(P10-Pad1)")
+    (add_net "Net-(P10-Pad2)")
+    (add_net "Net-(P10-Pad3)")
+    (add_net "Net-(P10-Pad4)")
     (add_net RF+)
     (add_net SCL2)
@@
     (pad 2 thru_hole oval (at 2.54 0 90) (size 1.7272 2.6) (drill 1.2) (layers *.Cu *.Mask)
       (net 10 GND))
+  )
+  (module Pin_Headers:Pin_Header_Straight_1x04_Pitch2.00mm (layer F.Cu)
+    (at 121.92 60.96 270)
+    (descr "Through hole pin header, 1x04, 2.00mm pitch, single row")
+    (tags "pin header single row")
+    (fp_text reference P9 (at 0.127 -2.54 270) (layer F.SilkS)
+      (effects (font (size 1 1) (thickness 0.15)))
+    )
+    (fp_text value CONN_01X04 (at 2.54 2.921 540) (layer F.Fab)
+      (effects (font (size 1 1) (thickness 0.15)))
+    )
+    (fp_line (start -1 1) (end 1 1) (layer F.SilkS) (width 0.15))
+    (fp_line (start 1 1) (end 1 7) (layer F.SilkS) (width 0.15))
+    (fp_line (start 1 7) (end -1 7) (layer F.SilkS) (width 0.15))
+    (fp_line (start -1 7) (end -1 1) (layer F.SilkS) (width 0.15))
+    (fp_line (start -1.6 -1.6) (end 1.6 -1.6) (layer F.CrtYd) (width 0.05))
+    (fp_line (start 1.6 -1.6) (end 1.6 7.6) (layer F.CrtYd) (width 0.05))
+    (fp_line (start 1.6 7.6) (end -1.6 7.6) (layer F.CrtYd) (width 0.05))
+    (fp_line (start -1.6 7.6) (end -1.6 -1.6) (layer F.CrtYd) (width 0.05))
+    (fp_line (start -1.5 0) (end -1.5 -1.5) (layer F.SilkS) (width 0.15))
+    (fp_line (start -1.5 -1.5) (end 0 -1.5) (layer F.SilkS) (width 0.15))
+    (pad 1 thru_hole rect (at 0 0 270) (size 1.35 1.016) (drill 0.8) (layers *.Cu *.Mask)
+      (net 62 "Net-(P10-Pad1)"))
+    (pad 2 thru_hole oval (at 0 2 270) (size 1.35 1.016) (drill 0.8) (layers *.Cu *.Mask)
+      (net 63 "Net-(P10-Pad2)"))
+    (pad 3 thru_hole oval (at 0 4 270) (size 1.35 1.016) (drill 0.8) (layers *.Cu *.Mask)
+      (net 64 "Net-(P10-Pad3)"))
+    (pad 4 thru_hole oval (at 0 6 270) (size 1.35 1.016) (drill 0.8) (layers *.Cu *.Mask)
+      (net 65 "Net-(P10-Pad4)"))
+    (model Pin_Headers.3dshapes/Pin_Header_Straight_1x04_Pitch2.00mm.wrl
+      (at (xyz 0 0 0))
+      (scale (xyz 1 1 1))
+      (rotate (xyz 0 0 0))
+    )
+  )
+  (module Pin_Headers:Pin_Header_Straight_1x04_Pitch2.00mm (layer F.Cu)
+    (at 121.92 58.42 270)
+    (descr "Through hole pin header, 1x04, 2.00mm pitch, single row")
+    (tags "pin header single row")
+    (fp_text reference P10 (at -0.127 -2.54 270) (layer F.SilkS)
+      (effects (font (size 1 1) (thickness 0.15)))
+    )
+    (fp_text value CONN_01X04 (at 0 9.017 450) (layer F.Fab)
+      (effects (font (size 1 1) (thickness 0.15)))
+    )
+    (fp_line (start -1 1) (end 1 1) (layer F.SilkS) (width 0.15))
+    (fp_line (start 1 1) (end 1 7) (layer F.SilkS) (width 0.15))
+    (fp_line (start 1 7) (end -1 7) (layer F.SilkS) (width 0.15))
+    (fp_line (start -1 7) (end -1 1) (layer F.SilkS) (width 0.15))
+    (fp_line (start -1.6 -1.6) (end 1.6 -1.6) (layer F.CrtYd) (width 0.05))
+    (fp_line (start 1.6 -1.6) (end 1.6 7.6) (layer F.CrtYd) (width 0.05))
+    (fp_line (start 1.6 7.6) (end -1.6 7.6) (layer F.CrtYd) (width 0.05))
+    (fp_line (start -1.6 7.6) (end -1.6 -1.6) (layer F.CrtYd) (width 0.05))
+    (fp_line (start -1.5 0) (end -1.5 -1.5) (layer F.SilkS) (width 0.15))
+    (fp_line (start -1.5 -1.5) (end 0 -1.5) (layer F.SilkS) (width 0.15))
+    (pad 1 thru_hole rect (at 0 0 270) (size 1.35 1.016) (drill 0.8) (layers *.Cu *.Mask)
+      (net 62 "Net-(P10-Pad1)"))
+    (pad 2 thru_hole oval (at 0 2 270) (size 1.35 1.016) (drill 0.8) (layers *.Cu *.Mask)
+      (net 63 "Net-(P10-Pad2)"))
+    (pad 3 thru_hole oval (at 0 4 270) (size 1.35 1.016) (drill 0.8) (layers *.Cu *.Mask)
+      (net 64 "Net-(P10-Pad3)"))
+    (pad 4 thru_hole oval (at 0 6 270) (size 1.35 1.016) (drill 0.8) (layers *.Cu *.Mask)
+      (net 65 "Net-(P10-Pad4)"))
+    (model Pin_Headers.3dshapes/Pin_Header_Straight_1x04_Pitch2.00mm.wrl
+      (at (xyz 0 0 0))
+      (scale (xyz 1 1 1))
+      (rotate (xyz 0 0 0))
+    )
+  )
+  (module Pin_Headers:Pin_Header_Straight_1x04_Pitch2.00mm (layer F.Cu)
+    (at 121.92 55.88 270)
+    (descr "Through hole pin header, 1x04, 2.00mm pitch, single row")
+    (tags "pin header single row")
+    (fp_text reference P11 (at -0.381 -2.54 270) (layer F.SilkS)
+      (effects (font (size 1 1) (thickness 0.15)))
+    )
+    (fp_text value CONN_01X04 (at -2.413 3.048 540) (layer F.Fab)
+      (effects (font (size 1 1) (thickness 0.15)))
+    )
+    (fp_line (start -1 1) (end 1 1) (layer F.SilkS) (width 0.15))
+    (fp_line (start 1 1) (end 1 7) (layer F.SilkS) (width 0.15))
+    (fp_line (start 1 7) (end -1 7) (layer F.SilkS) (width 0.15))
+    (fp_line (start -1 7) (end -1 1) (layer F.SilkS) (width 0.15))
+    (fp_line (start -1.6 -1.6) (end 1.6 -1.6) (layer F.CrtYd) (width 0.05))
+    (fp_line (start 1.6 -1.6) (end 1.6 7.6) (layer F.CrtYd) (width 0.05))
+    (fp_line (start 1.6 7.6) (end -1.6 7.6) (layer F.CrtYd) (width 0.05))
+    (fp_line (start -1.6 7.6) (end -1.6 -1.6) (layer F.CrtYd) (width 0.05))
+    (fp_line (start -1.5 0) (end -1.5 -1.5) (layer F.SilkS) (width 0.15))
+    (fp_line (start -1.5 -1.5) (end 0 -1.5) (layer F.SilkS) (width 0.15))
+    (pad 1 thru_hole rect (at 0 0 270) (size 1.35 1.016) (drill 0.8) (layers *.Cu *.Mask)
+      (net 62 "Net-(P10-Pad1)"))
+    (pad 2 thru_hole oval (at 0 2 270) (size 1.35 1.016) (drill 0.8) (layers *.Cu *.Mask)
+      (net 63 "Net-(P10-Pad2)"))
+    (pad 3 thru_hole oval (at 0 4 270) (size 1.35 1.016) (drill 0.8) (layers *.Cu *.Mask)
+      (net 64 "Net-(P10-Pad3)"))
+    (pad 4 thru_hole oval (at 0 6 270) (size 1.35 1.016) (drill 0.8) (layers *.Cu *.Mask)
+      (net 65 "Net-(P10-Pad4)"))
+    (model Pin_Headers.3dshapes/Pin_Header_Straight_1x04_Pitch2.00mm.wrl
+      (at (xyz 0 0 0))
+      (scale (xyz 1 1 1))
+      (rotate (xyz 0 0 0))
+    )
   )
   (gr_line (start 182.88 152.262735) (end 182.88 152.4) (layer Eco1.User) (width 0.2))
@@
   (segment (start 99.06 85.09) (end 99.06 90.17) (width 1.016) (layer B.Cu) (net 60) (status 30))
   (segment (start 68.58 70.485) (end 68.58 76.2) (width 1.016) (layer B.Cu) (net 61) (status 30))
+  (segment (start 121.92 58.42) (end 121.92 60.96) (width 1.016) (layer B.Cu) (net 62))
+  (segment (start 121.92 55.88) (end 121.92 58.42) (width 1.016) (layer B.Cu) (net 62))
+  (segment (start 119.92 58.42) (end 119.92 55.88) (width 1.016) (layer B.Cu) (net 63))
+  (segment (start 119.92 60.96) (end 119.92 58.42) (width 1.016) (layer B.Cu) (net 63))
+  (segment (start 117.92 58.42) (end 117.92 60.96) (width 1.016) (layer B.Cu) (net 64))
+  (segment (start 117.92 55.88) (end 117.92 58.42) (width 1.016) (layer B.Cu) (net 64))
+  (segment (start 115.92 58.42) (end 115.92 55.88) (width 1.016) (layer B.Cu) (net 65))
+  (segment (start 115.92 60.96) (end 115.92 58.42) (width 1.016) (layer B.Cu) (net 65))
   (zone (net 10) (net_name GND) (layer B.Cu) (hatch edge 0.508)
     (connect_pads yes (clearance 0.79248))

Commit message: First revision export
Parts:
- added C3: 0.1uF, Capacitors_THT:C_Disc_D3_P2.5, F.Cu at (94.0, 76.2)
- moved U2 5.08 mm to (66.0, 66.7)
- moved P7 5.08 mm to (73.7, 76.2)
- moved P10 2.54 mm to (121.9, 61.0)
- moved P11 2.54 mm to (121.9, 58.4)
- moved P9 2.54 mm to (121.9, 63.5)
Routing:
- net GND: track 16.5 -> 31.1 mm
- net +5V: track 58.6 -> 55.0 mm
- net TX_EN: track 20.7 -> 20.4 mm, vias 0 -> 2
- net (no net): vias 0 -> 4
Other:
- net class Default: clearance 0.79375 -> 0.8128
- net class Mounting Holes: clearance 0.79375 -> 0.8128
- net class Power: clearance 0.79375 -> 0.8128
- net class Signal: clearance 0.79375 -> 0.8128
- rule trace_clearance: 0.79375 -> 0.8128
